File: electronics/power-distribution-board/power-distribution-board.kicad_sch (KiCad schematic)
At the start: 17 parts

Commit message: merge electronics V1.x
Parts:
- removed C?: C, symbol Device:C
- removed J?: Conn_01x01, symbol Connector_Generic:Conn_01x01
- removed J? (x7): Conn_01x02, symbol Connector_Generic:Conn_01x02
- removed R?: R, symbol Device:R
- added C1: 10u/50V, Capacitor_SMD:C_1206_3216Metric, symbol Device:C
- added C2: 22u/25V, Capacitor_SMD:C_1206_3216Metric, symbol Device:C
- added C3: 150p, Capacitor_SMD:C_0603_1608Metric, symbol Device:C
- added C31: 1000u/50V, symbol Device:C_Polarized
- added C4, C5: 100n, Capacitor_SMD:C_0603_1608Metric, symbol Device:C
- added D1: SS36A, Diode_SMD:D_SMA, symbol Device:D_Schottky
- added H1, H2, H3, H4: MountingHole_Pad, MountingHole:MountingHole_3.2mm_M3_Pad_Via, symbol Mechanical:MountingHole_Pad
- added J4, J6, J7, J8, J9: Conn_01x02, goose:tht_pin_01x02, symbol Connector_Generic:Conn_01x02
- added J5: Conn_01x03, goose:tht_pin_01x03, symbol Connector_Generic:Conn_01x03
- added L1: 22u, Inductor_SMD:L_12x12mm_H6mm, symbol Device:L
- added R1, R32, R34: 210k, Resistor_SMD:R_0603_1608Metric, symbol Device:R
- added R2: 39k, Resistor_SMD:R_0603_1608Metric, symbol Device:R
- added R3, R4: 100k, Resistor_SMD:R_0603_1608Metric, symbol Device:R
- added R31, R33: 4k7, Resistor_SMD:R_0603_1608Metric, symbol Device:R
- added R35: 1m, Resistor_SMD:R_2512_6332Metric, symbol Device:R
- added U1: MP1584, Package_SO:SOIC-8-1EP_3.9x4.9mm_P1.27mm_EP2.62x3.51mm_ThermalVias, symbol goose:MP1584
- added U3: LM258, Package_SO:SOIC-8_3.9x4.9mm_P1.27mm, symbol Amplifier_Operational:LM358
- D11: renamed from D?; footprint (none) -> LED_SMD:LED_0603_1608Metric
- J1: renamed from J?; footprint (none) -> Connector_AMASS:AMASS_XT60-M_1x02_P7.20mm_Vertical
- J2: renamed from J?; footprint (none) -> goose:tht_pin_01x02
- R11: renamed from R?; value R -> 470k; footprint (none) -> Resistor_SMD:R_0603_1608Metric
- R12: renamed from R?; value R -> 100k; footprint (none) -> Resistor_SMD:R_0603_1608Metric
- R13: renamed from R?; footprint (none) -> Resistor_SMD:R_0603_1608Metric
- gave numbers to parts that had none: 1
Connections:
- net +3.3V is gone; now on net +5V: R13.1
- net +5V: now also C2.2, C5.2, J4.1 (Pin_1), J6.1 (Pin_1), J7.1 (Pin_1), J8.1 (Pin_1), J9.1 (Pin_1), L1.2, R1.2, U3.8 (V+)
- net +BATT: now also J3.2 (Pin_2), C1.2, R33.1, R35.1, U1.7 (VIN); no longer J1.1 (Pin_1), J3.1 (Pin_1), R11.1
- net GND: now also J1.1 (Pin_1), J3.1 (Pin_1), C1.1, C2.1, C31.2, C5.1, D1.2 (A), J4.2 (Pin_2), J5.3 (Pin_3), J6.2 (Pin_2), J7.2 (Pin_2), J8.2 (Pin_2), J9.2 (Pin_2), R2.1, R3.2, R32.1, R4.2, U1.5 (GND), U3.4 (V-); no longer J1.2 (Pin_2), J3.2 (Pin_2)
- net BATT_V_SENSE: now reaches R11.2, R12.1
- net BATT_V_SENSE: now also J5.2 (Pin_2)
- new net: R31.1, R32.2, U3.3 (+)
- new net: C3.2, R3.1
- new net: R33.2, R34.1, U3.2 (-)
- new net BATT_IN: C31.1, J1.2 (Pin_2), R11.1, R31.2, R35.2
- new net BATT_I_SENSE: J5.1 (Pin_1), R34.2, U3.1
- new net BST: C4.1, U1.8 (BST)
- new net COMP: C3.1, U1.3 (COMP)
- new net FB: R1.1, R2.2, U1.4 (FB)
- new net FREQ: R4.1, U1.6 (FREQ)
- new net SW: C4.2, D1.1 (K), L1.1, U1.1 (SW)
- no-connect marks 0 -> 5
Other:
- note added: "battery voltage measurement"
- note added: "current consumption measurement"
- note added: "current sense gain calculations: for: R31 = R33 R32 = R34 Vout = (R34/R33) * Rshunt*Ibatt R34 = (Vout * R33)/(Rshunt*Ibatt) assume: Ibatt = 70 A Rshunt = 0.001 ohm Vout = 3.1 V R33 = 4.7 kohm then: R34 = (3.1 * 4700)/(0.001*70) = 210 kohm"
- note added: "led resistor calculations: I_d = (U - U_f)/R13 R13 = (U - U_f)/I_d assume: I_d = 4 mA U_f = 1 V U = 5 V then: R13 = (5 - 1)/0.004 = 1 kohm"
- note added: "shunt resistor power calculations: Pshunt = Rshunt * I^2 assume: Rshunt = 0.001 ohm I = 50 A then: Pshunt = 0.001 * 50^2 = 2.5 W for 2512 resistor: Pmax = 3 W"
- note added: "voltage divider calcualtions: U_out = U_in * R12/(R11 + R12) U_out * (R11 + R12) = U_in * R12 U_out * R11 + U_out * R12 = U_in * R12 U_out * R11 = R12 * (U_in - U_out) R11 = R12 * (U_in - U_out)/U_out assume: R12 = 100 kohm U_in = 16.8 V U_out = 3.0 V then: R11 = 100k * (16.8-3)/3 = 470 kohm"
- note removed: "3.3V STEP-DOWN converter"
- note removed: "supply voltage measurement"
- moved on the sheet: D11, J1, J2, J3, R11, R12, R13
