File: electronics/wifi-receiver-transmitter/wifi-receiver-transmitter.kicad_pcb (KiCad board)
At the start: 2 copper layers, 38 x 38 mm, 34 parts, among them J1 Conn_01x02, J2 USB_B_Micro, J3 Conn_01x04, J4 Conn_01x06, Q1 Q_NPN_EBC, Q2 Q_NPN_EBC, SW1 SW_Push, SW2 SW_Push, U1 LM1117-3.3, U2 ESP-12E, U3 CH340G

Commit message: update esp module
Parts:
- removed the C6 at (145.2, 125.2)
- removed D1: BAT54C, Package_TO_SOT_SMD:SOT-23
- removed the J1 at (132.1, 119.4)
- added J3: Conn_01x04, goose:tht_pin_01x04, F.Cu at (132.2, 115.4)
- J1: renamed from J2; footprint Connector_USB:USB_Micro-B_Amphenol_10118194_Horizontal -> goose:usb_micro_B_druk_II
- R1, R2, R3, R4, R5, R8, R9: value 10k -> 4k7
- U3: value CH340G -> CH340C
- moved J4 33.9 mm to (166.0, 103.2)
- moved J2 33.5 mm to (132.2, 103.2)
- moved R6 25.4 mm to (136.8, 106.2), turned to 180 degrees
- moved R7 25.4 mm to (136.8, 108.2), turned to 180 degrees
- moved Q1 14.8 mm to (147.5, 114.5), turned to 180 degrees
- moved R8 12.5 mm to (151.8, 113.2), turned to 180 degrees
- moved C3 12.4 mm to (147.8, 119.5)
- moved C1 11.3 mm to (147.0, 122.0)
- moved C4 10.0 mm to (136.8, 110.2), turned to 180 degrees
- moved Q2 9.96 mm to (156.0, 114.5), turned to 0 degrees
- moved R9 9.86 mm to (151.8, 115.8), turned to 0 degrees
- moved C6 8.38 mm to (143.2, 113.0), turned to 0 degrees
- moved C7 8.13 mm to (163.8, 118.2), turned to 180 degrees
- moved G*** 6.94 mm to (151.6, 117.5)
- moved C5 6.54 mm to (142.5, 115.5), turned to 0 degrees
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- renumbered C7 to C2, C2 to C3, C5 to C4, C3 to C5, C4 to C6, C8 to C7, J3 to J2, U2 to U1, U1 to U2
Connections:
- C1 pad 1: /LDO_IN -> VBUS
- C2 pad 1: +5V -> +3.3V
- C3 pad 1: /LDO_IN -> VBUS
- C4 pad 1: +5V -> +3.3V
- U2 pad 3: /LDO_IN -> VBUS
Routing:
- net /GPIO1_TXD0: track 35.1 -> 67.2 mm
- net /GPIO3_RXD0: track 31.4 -> 63.3 mm, vias 2 -> 4
- net /RST: track 80.7 -> 50.1 mm, vias 4 -> 2
- net /GPIO4_SDA: track 17.5 -> 35.2 mm
- net +5V: track 16.1 -> 0.00 mm
- net /GPIO5_SCL: track 18.3 -> 34.3 mm
- net /LDO_IN: track 14.2 -> 0.00 mm
- net /DTR: track 25.9 -> 14.3 mm
- net unconnected-(J1-Pad6): track 11.5 -> 0.00 mm
- net /GPIO13_MOSI: track 17.0 -> 27.2 mm
- net /GPIO12_MISO: track 16.8 -> 27.0 mm
- net /GPIO14_SCLK: track 16.6 -> 26.8 mm
- net +3.3V: track 124.1 -> 114.4 mm, vias 10 -> 2
- net /RTS: track 26.5 -> 16.9 mm
- net VBUS: track 8.81 -> 18.2 mm
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Other:
- board text added: "GPIO1 TXD0"
- board text added: "GPIO15 CS"
- board text added: "GPIO3 RXD0"
- board text added: "UAV TVC Goose WiFi Recv-Transmit V1.1 by Eryk Możdżeń January 2023"
- board text removed: "GPIO15 CS TXD2"
- board text removed: "UAV TVC Goose WiFi Recv-Transmit V1.0 by Eryk Możdżeń December 2022"
- board text removed: "VIN"
