File: electronics/wifi-receiver-transmitter/wifi-receiver-transmitter.kicad_sch (KiCad schematic)
At the start: 9 parts

Commit message: merge electronics V1.x
Parts:
- removed C?: 100n, symbol Device:C
- added C1, C4, C5, C6, C8: 100n, Capacitor_SMD:C_0603_1608Metric, symbol Device:C
- added C2, C3, C7: 4u7, Capacitor_Tantalum_SMD:CP_EIA-3216-18_Kemet-A, symbol Device:C_Polarized
- added D1: BAT54C, Package_TO_SOT_SMD:SOT-23, symbol Diode:BAT54C
- added H1, H2, H3, H4: MountingHole_Pad, MountingHole:MountingHole_3.2mm_M3_Pad_Via, symbol Mechanical:MountingHole_Pad
- added J1: Conn_01x02, goose:tht_pin_01x02, symbol Connector_Generic:Conn_01x02
- added J2: USB_B_Micro, Connector_USB:USB_Micro-B_Amphenol_10118194_Horizontal, symbol Connector:USB_B_Micro
- added J3: Conn_01x04, goose:tht_pin_01x04, symbol Connector_Generic:Conn_01x04
- added J4: Conn_01x06, goose:tht_pin_01x06, symbol Connector_Generic:Conn_01x06
- added Q1, Q2: Q_NPN_EBC, Package_TO_SOT_SMD:SOT-23, symbol Device:Q_NPN_EBC
- added R6, R7, R8, R9: 4k7, Resistor_SMD:R_0603_1608Metric, symbol Device:R
- added U1: LM1117-3.3, Package_TO_SOT_SMD:SOT-223-3_TabPin2, symbol Regulator_Linear:LM1117-3.3
- added U3: CH340G, Package_SO:SOIC-16_3.9x9.9mm_P1.27mm, symbol Interface_USB:CH340G
- R1, R2, R3, R4, R5: renamed from R?; value 10k -> 4k7; footprint (none) -> Resistor_SMD:R_0603_1608Metric
- SW1, SW2: renamed from SW?; footprint (none) -> Button_Switch_SMD:SW_Push_SPST_NO_Alps_SKRK
- gave numbers to parts that had none: 1
Connections:
- net +3.3V: now also C3.1, C4.1, C8.1, J3.4 (Pin_4), J4.6 (Pin_6), R6.1, R7.1, U1.2 (VO), U3.16 (VCC), U3.4 (V3)
- net GND: now also C1.2, C2.2, C3.2, C4.2, C5.2, C6.2, C7.2, C8.2, J1.1 (Pin_1), J2.5 (GND), J3.1 (Pin_1), J4.1 (Pin_1), U1.1 (GND), U3.1 (GND)
- net GPIO0_FLASH: now reaches R4.2, SW2.2, U2.18 (GPIO0)
- net GPIO0_FLASH: now also Q2.3 (C)
- net RST: now reaches R2.2, SW1.2, U2.1 (~{RST})
- net RST: now also Q1.3 (C)
- net EN: now reaches R1.2, U2.3 (EN)
- net GPIO15_CS_TXD2: now reaches R3.1, U2.16 (GPIO15)
- net GPIO15_CS_TXD2: now also J4.5 (Pin_5)
- net GPIO2_TXD1: now reaches R5.2, U2.17 (GPIO2)
- net GPIO4_SDA: now reaches U2.19 (GPIO4)
- net GPIO4_SDA: now also J3.2 (Pin_2), R7.2
- net ADC: now reaches U2.2 (ADC)
- net GPIO5_SCL: now reaches U2.20 (GPIO5)
- net GPIO5_SCL: now also J3.3 (Pin_3), R6.2
- net GPIO16_WAKE: now reaches U2.4 (GPIO16)
- net GPIO14_SCLK: now reaches U2.5 (GPIO14)
- net GPIO14_SCLK: now also J4.4 (Pin_4)
- net GPIO12_MISO: now reaches U2.6 (GPIO12)
- net GPIO12_MISO: now also J4.3 (Pin_3)
- net GPIO13_MOSI: now reaches U2.7 (GPIO13)
- net GPIO13_MOSI: now also J4.2 (Pin_2)
- net RXD renamed GPIO3_RXD0
- net GPIO3_RXD0: now also U3.2 (TXD)
- net TXD renamed GPIO1_TXD0
- net GPIO1_TXD0: now also U3.3 (RXD)
- new net: Q1.2 (B), R8.2
- new net: Q2.2 (B), R9.2
- new net +5V: C5.1, C7.1, D1.1, J1.2 (Pin_2)
- new net D+: J2.3 (D+), U3.5 (UD+)
- new net D-: J2.2 (D-), U3.6 (UD-)
- new net DTR: Q2.1 (E), R8.1, U3.13 (~{DTR})
- new net LDO_IN: C1.1, C2.1, D1.3, U1.3 (VI)
- new net RTS: Q1.1 (E), R9.1, U3.14 (~{RTS})
- new net VBUS: C6.1, D1.2, J2.1 (VBUS)
- no-connect marks 6 -> 19
Other:
- note added: "LDO regulator"
- note added: "USB/UART converter"
- note added: "connectors"
- note added: "twisted"
- moved on the sheet: R1, R2, R3, R4, R5, SW1, SW2, U2

Commit message: update esp module
Parts:
- removed C6: 100n, Capacitor_SMD:C_0603_1608Metric, symbol Device:C
- removed D1: BAT54C, Package_TO_SOT_SMD:SOT-23, symbol Diode:BAT54C
- removed J1: Conn_01x02, goose:tht_pin_01x02, symbol Connector_Generic:Conn_01x02
- removed U3: CH340G, Package_SO:SOIC-16_3.9x9.9mm_P1.27mm, symbol Interface_USB:CH340G
- added J3: Conn_01x04, goose:tht_pin_01x04, symbol Connector_Generic:Conn_01x04
- added U3: CH340C, Package_SO:SOIC-16_3.9x9.9mm_P1.27mm, symbol Interface_USB:CH340C
- J1: renamed from J2; footprint Connector_USB:USB_Micro-B_Amphenol_10118194_Horizontal -> goose:usb_micro_B_druk_II
- renumbered C7 to C2, C2 to C3, C5 to C4, C3 to C5, C4 to C6, C8 to C7, J3 to J2, U2 to U1, U1 to U2
Connections:
- net +5V is gone; now on net +3.3V: C2.1, C4.1
- net LDO_IN is gone; now on net VBUS: C1.1, C3.1, U2.3 (VI)
- net +3.3V: now also J3.4 (Pin_4), U3.16 (VCC), U3.4 (V3)
- net D+: now also U3.5 (UD+)
- net D-: now also U3.6 (UD-)
- net DTR: now also U3.13 (~{DTR})
- net GND: now also J3.1 (Pin_1), U3.1 (GND)
- net GPIO1_TXD0: now also J3.3 (Pin_3), U3.3 (RXD)
- net GPIO3_RXD0: now also J3.2 (Pin_2), U3.2 (TXD)
- net RTS: now also U3.14 (~{RTS})
- no-connect marks 19 -> 17
Other:
- moved on the sheet: C1, C2, C3, C4, C5, C6, H1, H2, H3, H4, J2, J4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
