File: electronics/flight-controller/flight-controller.kicad_sch (KiCad schematic)
At the start: 30 parts

Commit message: merge electronics V1.x
Parts:
- removed C? (x11): 100n, symbol Device:C
- removed C? (x2): 22p, symbol Device:C
- removed C?: 1u, symbol Device:C
- removed C?: 2n2, symbol Device:C
- removed C?: 2u2, symbol Device:C
- removed C?: 4.7u, symbol Device:C
- removed L?: 4.7u, symbol Device:L
- removed R? (x6): 4k7, symbol Device:R
- removed R?: 10k, symbol Device:R
- removed SW?: SW_Push, symbol Switch:SW_Push
- removed U?: STM32F411RETx, Package_QFP:LQFP-64_10x10mm_P0.5mm, symbol MCU_ST_STM32F4:STM32F411RETx
- removed U?: BMP280, Package_LGA:Bosch_LGA-8_2x2.5mm_P0.65mm_ClockwisePinNumbering, symbol Sensor_Pressure:BMP280
- removed U?: MPU-6050, Sensor_Motion:InvenSense_QFN-24_4x4mm_P0.5mm, symbol Sensor_Motion:MPU-6050
- removed Y?: 8MHz, symbol Device:Crystal
- added H1, H2, H3, H4: MountingHole_Pad, MountingHole:MountingHole_3.2mm_M3_Pad_Via, symbol Mechanical:MountingHole_Pad
Connections:
- no-connect marks 2 -> 4
Other:
- added sheet power (power.kicad_sch)
- added sheet sensors (sensors.kicad_sch)
- added sheet ucontroller (ucontroller.kicad_sch)
- note removed: "I2C address: 0b1101000 0x68"
- note removed: "I2C address: 0b1110111 0x77"
- note removed: "IMU"
- note removed: "barometer"
- note removed: "uController"
