File: electronics/flight-controller/sensors.kicad_sch (KiCad schematic)
At the start: 12 parts, among them U3 BMP280, U4 MPU-6050, U5 QMC5883L

Commit message: barometer and magnetometer works
Parts:
- U5: value QMC5883L -> HMC5883L
Other:
- note added: "I2C address: 0x1E"
- note removed: "I2C address: 0b0001101 0x0D"
Changed lines of the file:
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@@
     (effects (font (size 1.27 1.27) (thickness 0.254) bold) (justify left bottom))
   )
-  (text "I2C address:\n0b0001101\n0x0D" (at 180.34 85.09 0)
+  (text "I2C address:\n0x1E" (at 180.34 85.09 0)
     (effects (font (size 1.27 1.27) (thickness 0.254) bold) (justify left bottom))
   )
@@
       (effects (font (size 1.27 1.27)) (justify left))
     )
-    (property "Value" "QMC5883L" (id 1) (at 210.82 81.28 0)
+    (property "Value" "HMC5883L" (id 1) (at 210.82 81.28 0)
       (effects (font (size 1.27 1.27)) (justify left))
     )
