File: electronics_v2/flight-controller-v2/flight-controller-v2.kicad_pcb (KiCad board)
At the start: 4 copper layers, 45 x 89 mm, 114 parts, among them J1 Conn_01x02, J10 Conn_01x05, J12 Conn_02x03_Odd_Even, J2 Conn_01x03, J3 Conn_01x03, J4 Conn_01x03, J5 Conn_01x03, J6 Conn_01x03, J7 Conn_01x02, J8 USB_B_Micro, J9 Conn_01x06, Q1 IRFR5305, SW1 SW_Push_SPDT, SW2 SW_Push, SW3 SW_Push, U1 LM1117-3.3, U10 HMC5883L, U2 MP1584, U3 INA226, U4 STM32F411RETx, U5 ESP-12E, U6 BMP280, U7 CS49E, U8 MPU-6050, U9 LM393, Y1 8MHz

Commit message: route new FC
Parts:
- added J11: Conn_01x06, goose:tht_pin_01x06, F.Cu at (141.2, 96.8)
- C15, C19: moved to F.Cu
- D1: value RED -> LED
- J9: value Conn_01x06 -> Conn_01x05; footprint goose:tht_pin_01x06 -> goose:tht_pin_01x05
- R13: value 210k -> 200k
- moved G*** 65.9 mm to (165.0, 145.2)
- moved J10 29.9 mm to (159.3, 77.5), turned to 90 degrees
- moved C13 20.8 mm to (134.8, 99.5)
- moved C19 20.5 mm to (126.2, 116.8), turned to 180 degrees
- moved Y1 19.5 mm to (134.8, 100.4), turned to 180 degrees
- moved C11 18.1 mm to (134.8, 101.5)
- moved R18 15.5 mm to (134.8, 116.2)
- moved C15 14.7 mm to (126.2, 118.8), turned to 0 degrees
- moved D5 11.9 mm to (137.5, 122.2)
- moved D3 11.7 mm to (137.5, 118.2)
- moved R22 11.5 mm to (134.8, 114.2)
- moved D4 11.1 mm to (137.5, 120.2)
- moved C16 11.0 mm to (134.8, 110.2)
- moved R24 10.9 mm to (138.2, 106.2), turned to 180 degrees
- moved C21 8.27 mm to (138.2, 116.2)
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Connections:
- J9 pad 1: /ucontroller/PA0 -> /ucontroller/SPI3_SCK
- J9 pad 2: GND -> +3.3V
- J9 pad 3: /ucontroller/UART2_TX -> /ucontroller/SPI3_MISO
- J9 pad 4: /ucontroller/UART2_RX -> /ucontroller/SPI3_MOSI
- J9 pad 5: +3.3V -> GND
- U4 pad 2: /sensors/VLX_XSHUT -> unconnected-(U4-Pad2)
- U4 pad 3: /sensors/VLX_INT -> unconnected-(U4-Pad3)
- U4 pad 39: unconnected-(U4-Pad39) -> /sensors/VLX_XSHUT
- U4 pad 43: unconnected-(U4-Pad43) -> /sensors/VLX_INT
- U4 pad 50: /sensors/IMU_INT -> unconnected-(U4-Pad50)
- U4 pad 51: unconnected-(U4-Pad51) -> /ucontroller/SPI3_SCK
- U4 pad 52: unconnected-(U4-Pad52) -> /ucontroller/SPI3_MISO
- U4 pad 53: unconnected-(U4-Pad53) -> /ucontroller/SPI3_MOSI
- U4 pad 56: unconnected-(U4-Pad56) -> /sensors/IMU_INT
Routing:
- net GND: track 0.00 -> 105.0 mm, vias 0 -> 97
- net /ucontroller/RESET: track 0.00 -> 98.4 mm, vias 0 -> 4
- net /ucontroller/SWDIO: track 0.00 -> 74.3 mm, vias 0 -> 5
- net /ucontroller/SWCLK: track 0.00 -> 68.1 mm, vias 0 -> 5
- net +3.3V: track 0.00 -> 62.2 mm, vias 0 -> 46
- net +5V: track 0.00 -> 56.1 mm, vias 0 -> 35
- net /power/PWM_SERVO4: track 0.00 -> 48.5 mm, vias 0 -> 1
- net /sensors/HALL: track 0.00 -> 47.8 mm, vias 0 -> 2
- net /power/PWM_SERVO3: track 0.00 -> 47.4 mm, vias 0 -> 1
- net /power/INT_I2C_SCL: track 0.00 -> 45.9 mm, vias 0 -> 5
- net /ucontroller/ESP_UART1_RX: track 0.00 -> 44.7 mm, vias 0 -> 3
- net /power/INT_I2C_SDA: track 0.00 -> 42.2 mm, vias 0 -> 5
- net /power/PWM_SERVO2: track 0.00 -> 41.4 mm, vias 0 -> 1
- net /ucontroller/SPI3_SCK: track 0.00 -> 40.6 mm, vias 0 -> 2
- net /ucontroller/ESP_UART1_TX: track 0.00 -> 39.4 mm, vias 0 -> 3
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- added copper zone on F.Cu, net +3.3V
- added copper zone on B.Cu, net +5V
- added copper zone on F.Cu, net +5V
- added copper zone on In2.Cu, net +5V
- added copper zone on F.Cu, net /power/SW
- added copper zone on B.Cu, net GND
Other:
- board text added: "MISO"
- board text added: "MOSI"
- board text added: "SCK"
