File: electronics_v2/flight-controller-v2/ucontroller.kicad_sch (KiCad schematic)
At the start: 45 parts, among them J10 Conn_01x05, J8 USB_B_Micro, J9 Conn_01x06, SW2 SW_Push, SW3 SW_Push, U4 STM32F411RETx, U5 ESP-12E, Y1 8MHz

Commit message: route new FC
Parts:
- added J9: Conn_01x05, goose:tht_pin_01x05, symbol Connector_Generic:Conn_01x05
- renumbered J9 to J11
Connections:
- net +3.3V: now also J11.2 (Pin_2), J9.2 (Pin_2); no longer J11.5 (Pin_5)
- net GND: now also J11.5 (Pin_5), J9.5 (Pin_5); no longer J11.2 (Pin_2)
- net IMU_INT: now also U4.56 (PB4); no longer U4.50 (PA15)
- net UART2_RX: now also J11.3 (Pin_3); no longer J11.4 (Pin_4)
- net UART2_TX: now also J11.4 (Pin_4); no longer J11.3 (Pin_3)
- net VLX_INT: now also U4.43 (PA10); no longer U4.3 (PC14)
- net VLX_XSHUT: now also U4.39 (PC8); no longer U4.2 (PC13)
- net SPI3_SCK: now reaches U4.51 (PC10)
- net SPI3_SCK: now also J9.1 (Pin_1)
- net SPI3_MISO: now reaches U4.52 (PC11)
- net SPI3_MISO: now also J9.3 (Pin_3)
- net SPI3_MOSI: now reaches U4.53 (PC12)
- net SPI3_MOSI: now also J9.4 (Pin_4)
- no-connect marks 34 -> 31
Other:
- moved on the sheet: J11
Changed lines of the file:
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@@
   )
   (no_connect (at 113.03 99.06))
-  (no_connect (at 113.03 134.62))
   (no_connect (at 77.47 124.46))
   (no_connect (at 113.03 132.08))
@@
   (no_connect (at 204.47 43.18))
   (no_connect (at 77.47 129.54))
-  (no_connect (at 113.03 106.68))
+  (no_connect (at 77.47 154.94))
+  (no_connect (at 77.47 157.48))
   (no_connect (at 113.03 91.44))
   (no_connect (at 201.93 130.81))
@@
   (no_connect (at 113.03 160.02))
   (no_connect (at 201.93 146.05))
-  (no_connect (at 77.47 152.4))
-  (no_connect (at 77.47 147.32))
-  (no_connect (at 77.47 149.86))
-  (no_connect (at 77.47 142.24))
   (no_connect (at 201.93 138.43))
+  (no_connect (at 113.03 119.38))
   (wire (pts (xy 140.97 101.6) (xy 144.78 101.6))
     (stroke (width 0) (type default) (color 0 0 0 0))
@@
     (effects (font (size 1.27 1.27) (thickness 0.254) bold) (justify left bottom))
   )
-  (label "UART2_RX" (at 196.85 76.2 180)
+  (label "SPI3_MISO" (at 201.93 76.2 180)
     (effects (font (size 1.27 1.27)) (justify right bottom))
   )
+  (label "UART2_RX" (at 252.73 73.66 180)
+    (effects (font (size 1.27 1.27)) (justify right bottom))
+  )
+  (label "SPI3_SCK" (at 77.47 147.32 180)
+    (effects (font (size 1.27 1.27)) (justify right bottom))
+  )
+  (label "SPI3_MOSI" (at 201.93 78.74 180)
+    (effects (font (size 1.27 1.27)) (justify right bottom))
+  )
   (label "PA0" (at 113.03 81.28 0)
     (effects (font (size 1.27 1.27)) (justify left bottom))
@@
   (label "ESP_GPIO12" (at 232.41 135.89 0)
     (effects (font (size 1.27 1.27)) (justify left bottom))
+  )
+  (label "SPI3_MISO" (at 77.47 149.86 180)
+    (effects (font (size 1.27 1.27)) (justify right bottom))
   )
   (label "ESP_GPIO1_TXD0" (at 232.41 123.19 0)
@@
     (effects (font (size 1.27 1.27)) (justify left bottom))
   )
-  (label "UART2_TX" (at 196.85 73.66 180)
+  (label "UART2_TX" (at 252.73 76.2 180)
     (effects (font (size 1.27 1.27)) (justify right bottom))
   )
@@
     (effects (font (size 1.27 1.27)) (justify left bottom))
   )
-  (label "PA0" (at 196.85 68.58 180)
+  (label "PA0" (at 252.73 68.58 180)
     (effects (font (size 1.27 1.27)) (justify right bottom))
   )
@@
   (label "USB_D-" (at 212.09 40.64 0)
     (effects (font (size 1.27 1.27)) (justify left bottom))
+  )
+  (label "SPI3_MOSI" (at 77.47 152.4 180)
+    (effects (font (size 1.27 1.27)) (justify right bottom))
   )
   (label "SWCLK" (at 252.73 39.37 180)
@@
     (effects (font (size 1.27 1.27)) (justify right bottom))
   )
-  (label "PA1" (at 196.85 81.28 180)
+  (label "PA1" (at 252.73 81.28 180)
     (effects (font (size 1.27 1.27)) (justify right bottom))
   )
@@
     (effects (font (size 1.27 1.27)) (justify right bottom))
   )
+  (label "SPI3_SCK" (at 201.93 71.12 180)
+    (effects (font (size 1.27 1.27)) (justify right bottom))
+  )
   (label "ESP_UART1_RX" (at 113.03 142.24 0)
     (effects (font (size 1.27 1.27)) (justify left bottom))
@@
     (effects (font (size 1.27 1.27)) (justify left))
   )
-  (hierarchical_label "IMU_INT" (shape input) (at 113.03 119.38 0)
+  (hierarchical_label "IMU_INT" (shape input) (at 113.03 134.62 0)
     (effects (font (size 1.27 1.27)) (justify left))
   )
@@
     (effects (font (size 1.27 1.27)) (justify left))
   )
-  (hierarchical_label "VLX_XSHUT" (shape output) (at 77.47 154.94 180)
+  (hierarchical_label "VLX_XSHUT" (shape output) (at 77.47 142.24 180)
     (effects (font (size 1.27 1.27)) (justify right))
   )
-  (hierarchical_label "VLX_INT" (shape input) (at 77.47 157.48 180)
-    (effects (font (size 1.27 1.27)) (justify right))
+  (hierarchical_label "VLX_INT" (shape input) (at 113.03 106.68 0)
+    (effects (font (size 1.27 1.27)) (justify left))
   )
   (symbol (lib_id "Device:R") (at 39.37 50.8 0) (unit 1)
@@
     )
     (property "Datasheet" "" (id 3) (at 196.85 48.26 0)
+      (effects (font (size 1.27 1.27)) hide)
+    )
+    (pin "1")
+  )
+  (symbol (lib_id "power:GND") (at 201.93 81.28 270) (unit 1)
+    (in_bom yes) (on_board yes)
+    (property "Reference" "#PWR059" (id 0) (at 195.58 81.28 0)
+      (effects (font (size 1.27 1.27)) hide)
+    )
+    (property "Value" "GND" (id 1) (at 198.12 81.28 90)
+      (effects (font (size 1.27 1.27)) (justify right))
+    )
+    (property "Footprint" "" (id 2) (at 201.93 81.28 0)
+      (effects (font (size 1.27 1.27)) hide)
+    )
+    (property "Datasheet" "" (id 3) (at 201.93 81.28 0)
+      (effects (font (size 1.27 1.27)) hide)
+    )
+    (pin "1")
+  )
+  (symbol (lib_id "power:+3.3V") (at 201.93 73.66 90) (unit 1)
+    (in_bom yes) (on_board yes)
+    (property "Reference" "#PWR058" (id 0) (at 205.74 73.66 0)
+      (effects (font (size 1.27 1.27)) hide)
+    )
+    (property "Value" "+3.3V" (id 1) (at 193.04 73.66 90)
+      (effects (font (size 1.27 1.27)) (justify right))
+    )
+    (property "Footprint" "" (id 2) (at 201.93 73.66 0)
+      (effects (font (size 1.27 1.27)) hide)
+    )
+    (property "Datasheet" "" (id 3) (at 201.93 73.66 0)
       (effects (font (size 1.27 1.27)) hide)
     )
@@
     (pin "1")
   )
-  (symbol (lib_id "power:GND") (at 196.85 71.12 270) (unit 1)
-    (in_bom yes) (on_board yes)
-    (property "Reference" "#PWR058" (id 0) (at 190.5 71.12 0)
-      (effects (font (size 1.27 1.27)) hide)
-    )
-    (property "Value" "GND" (id 1) (at 193.04 71.12 90)
+  (symbol (lib_id "power:GND") (at 252.73 78.74 270) (unit 1)
+    (in_bom yes) (on_board yes)
+    (property "Reference" "#PWR070" (id 0) (at 246.38 78.74 0)
+      (effects (font (size 1.27 1.27)) hide)
+    )
+    (property "Value" "GND" (id 1) (at 248.92 78.74 90)
       (effects (font (size 1.27 1.27)) (justify right))
     )
-    (property "Footprint" "" (id 2) (at 196.85 71.12 0)
-      (effects (font (size 1.27 1.27)) hide)
-    )
-    (property "Datasheet" "" (id 3) (at 196.85 71.12 0)
+    (property "Footprint" "" (id 2) (at 252.73 78.74 0)
+      (effects (font (size 1.27 1.27)) hide)
+    )
+    (property "Datasheet" "" (id 3) (at 252.73 78.74 0)
       (effects (font (size 1.27 1.27)) hide)
     )
@@
     (pin "2")
   )
-  (symbol (lib_id "power:+3.3V") (at 196.85 78.74 90) (unit 1)
-    (in_bom yes) (on_board yes)
-    (property "Reference" "#PWR059" (id 0) (at 200.66 78.74 0)
-      (effects (font (size 1.27 1.27)) hide)
-    )
-    (property "Value" "+3.3V" (id 1) (at 187.96 78.74 90)
+  (symbol (lib_id "power:+3.3V") (at 252.73 71.12 90) (unit 1)
+    (in_bom yes) (on_board yes)
+    (property "Reference" "#PWR069" (id 0) (at 256.54 71.12 0)
+      (effects (font (size 1.27 1.27)) hide)
+    )
+    (property "Value" "+3.3V" (id 1) (at 243.84 71.12 90)
       (effects (font (size 1.27 1.27)) (justify right))
     )
-    (property "Footprint" "" (id 2) (at 196.85 78.74 0)
-      (effects (font (size 1.27 1.27)) hide)
-    )
-    (property "Datasheet" "" (id 3) (at 196.85 78.74 0)
+    (property "Footprint" "" (id 2) (at 252.73 71.12 0)
+      (effects (font (size 1.27 1.27)) hide)
+    )
+    (property "Datasheet" "" (id 3) (at 252.73 71.12 0)
       (effects (font (size 1.27 1.27)) hide)
     )
@@
     (pin "2")
   )
-  (symbol (lib_id "Connector_Generic:Conn_01x06") (at 201.93 73.66 0) (unit 1)
-    (in_bom yes) (on_board yes) (fields_autoplaced)
-    (property "Reference" "J9" (id 0) (at 204.47 73.6599 0)
-      (effects (font (size 1.27 1.27)) (justify left))
-    )
-    (property "Value" "Conn_01x06" (id 1) (at 204.47 76.1999 0)
-      (effects (font (size 1.27 1.27)) (justify left))
-    )
-    (property "Footprint" "goose:tht_pin_01x06" (id 2) (at 201.93 73.66 0)
-      (effects (font (size 1.27 1.27)) hide)
-    )
-    (property "Datasheet" "~" (id 3) (at 201.93 73.66 0)
+  (symbol (lib_id "Connector_Generic:Conn_01x06") (at 257.81 73.66 0) (unit 1)
+    (in_bom yes) (on_board yes) (fields_autoplaced)
+    (property "Reference" "J11" (id 0) (at 260.35 73.6599 0)
+      (effects (font (size 1.27 1.27)) (justify left))
+    )
+    (property "Value" "Conn_01x06" (id 1) (at 260.35 76.1999 0)
+      (effects (font (size 1.27 1.27)) (justify left))
+    )
+    (property "Footprint" "goose:tht_pin_01x06" (id 2) (at 257.81 73.66 0)
+      (effects (font (size 1.27 1.27)) hide)
+    )
+    (property "Datasheet" "~" (id 3) (at 257.81 73.66 0)
       (effects (font (size 1.27 1.27)) hide)
     )
@@
   (symbol (lib_id "Device:R") (at 142.24 139.7 0) (unit 1)
     (in_bom yes) (on_board yes)
-    (property "Reference" "R23" (id 0) (at 138.43 138.43 0)
+    (property "Reference" "R23" (id 0) (at 137.16 138.43 0)
       (effects (font (size 1.27 1.27)) (justify left))
     )
@@
     (pin "2")
   )
+  (symbol (lib_id "Connector_Generic:Conn_01x05") (at 207.01 76.2 0) (unit 1)
+    (in_bom yes) (on_board yes)
+    (property "Reference" "J9" (id 0) (at 209.55 73.66 0)
+      (effects (font (size 1.27 1.27)) (justify left))
+    )
+    (property "Value" "Conn_01x05" (id 1) (at 209.55 76.2 0)
+      (effects (font (size 1.27 1.27)) (justify left))
+    )
+    (property "Footprint" "goose:tht_pin_01x05" (id 2) (at 207.01 76.2 0)
+      (effects (font (size 1.27 1.27)) hide)
+    )
+    (property "Datasheet" "~" (id 3) (at 207.01 76.2 0)
+      (effects (font (size 1.27 1.27)) hide)
+    )
+    (pin "1")
+    (pin "2")
+    (pin "3")
+    (pin "4")
+    (pin "5")
+  )
   (symbol (lib_id "power:GND") (at 72.39 101.6 0) (unit 1)
