File: electronics-v2/flight-controller-v2/power.kicad_sch (KiCad schematic)
At the start: 39 parts, among them J1 Conn_01x02, J2 Conn_01x03, J3 Conn_01x03, J4 Conn_01x03, J5 Conn_01x03, J6 Conn_01x03, J7 Conn_01x02, Q1 IRFR5305, SW1 SW_Push_SPDT, U1 LM1117-3.3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

Commit message: fixes in routing
Connections:
- net INT_I2C_SCL renamed SENSOR_I2C_SCL
- net INT_I2C_SDA renamed SENSOR_I2C_SDA
Changed lines of the file:
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@@
   (junction (at 144.78 49.53) (diameter 0) (color 0 0 0 0)
   )
-  (junction (at 240.03 39.37) (diameter 0) (color 0 0 0 0)
-  )
   (junction (at 171.45 97.79) (diameter 0) (color 0 0 0 0)
+  )
+  (junction (at 222.25 36.83) (diameter 0) (color 0 0 0 0)
   )
   (junction (at 199.39 49.53) (diameter 0) (color 0 0 0 0)
@@
     (stroke (width 0) (type default) (color 0 0 0 0))
   )
+  (wire (pts (xy 222.25 36.83) (xy 226.06 36.83))
+    (stroke (width 0) (type default) (color 0 0 0 0))
+  )
   (wire (pts (xy 153.67 39.37) (xy 144.78 39.37))
     (stroke (width 0) (type default) (color 0 0 0 0))
@@
     (stroke (width 0) (type default) (color 0 0 0 0))
   )
-  (wire (pts (xy 240.03 39.37) (xy 240.03 40.64))
-    (stroke (width 0) (type default) (color 0 0 0 0))
-  )
   (wire (pts (xy 166.37 90.17) (xy 166.37 97.79))
     (stroke (width 0) (type default) (color 0 0 0 0))
@@
     (stroke (width 0) (type default) (color 0 0 0 0))
   )
-  (wire (pts (xy 220.98 39.37) (xy 240.03 39.37))
+  (wire (pts (xy 220.98 39.37) (xy 222.25 39.37))
     (stroke (width 0) (type default) (color 0 0 0 0))
   )
@@
     (stroke (width 0) (type default) (color 0 0 0 0))
   )
-  (wire (pts (xy 240.03 36.83) (xy 240.03 39.37))
+  (wire (pts (xy 222.25 36.83) (xy 222.25 39.37))
     (stroke (width 0) (type default) (color 0 0 0 0))
   )
@@
     (stroke (width 0) (type default) (color 0 0 0 0))
   )
-  (wire (pts (xy 220.98 36.83) (xy 240.03 36.83))
+  (wire (pts (xy 226.06 36.83) (xy 226.06 38.1))
+    (stroke (width 0) (type default) (color 0 0 0 0))
+  )
+  (wire (pts (xy 220.98 36.83) (xy 222.25 36.83))
     (stroke (width 0) (type default) (color 0 0 0 0))
   )
@@
     (effects (font (size 1.27 1.27)) (justify right))
   )
-  (hierarchical_label "INT_I2C_SDA" (shape bidirectional) (at 220.98 44.45 0)
+  (hierarchical_label "SENSOR_I2C_SDA" (shape bidirectional) (at 220.98 44.45 0)
     (effects (font (size 1.27 1.27)) (justify left))
   )
@@
     (effects (font (size 1.27 1.27)) (justify right))
   )
-  (hierarchical_label "INT_I2C_SCL" (shape bidirectional) (at 220.98 46.99 0)
+  (hierarchical_label "SENSOR_I2C_SCL" (shape bidirectional) (at 220.98 46.99 0)
     (effects (font (size 1.27 1.27)) (justify left))
   )
@@
     (pin "1")
   )
-  (symbol (lib_id "power:GND") (at 240.03 40.64 0) (unit 1)
-    (in_bom yes) (on_board yes)
-    (property "Reference" "#PWR020" (id 0) (at 240.03 46.99 0)
-      (effects (font (size 1.27 1.27)) hide)
-    )
-    (property "Value" "GND" (id 1) (at 240.03 44.45 0))
-    (property "Footprint" "" (id 2) (at 240.03 40.64 0)
-      (effects (font (size 1.27 1.27)) hide)
-    )
-    (property "Datasheet" "" (id 3) (at 240.03 40.64 0)
-      (effects (font (size 1.27 1.27)) hide)
-    )
+  (symbol (lib_id "power:GND") (at 226.06 38.1 0) (unit 1)
+    (in_bom yes) (on_board yes)
+    (property "Reference" "#PWR020" (id 0) (at 226.06 44.45 0)
+      (effects (font (size 1.27 1.27)) hide)
+    )
+    (property "Value" "GND" (id 1) (at 226.06 41.91 0))
+    (property "Footprint" "" (id 2) (at 226.06 38.1 0)
+      (effects (font (size 1.27 1.27)) hide)
+    )
+    (property "Datasheet" "" (id 3) (at 226.06 38.1 0)
+      (effects (font (size 1.27 1.27)) hide)
+    )

Commit message: generate schematic
Other:
- title: (none) -> UAV TVC Goose Flight Controller
Changed lines of the file:
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@@
 (kicad_sch (version 20211123) (generator eeschema)
   (paper "A4")
+  (title_block
+    (title "UAV TVC Goose Flight Controller")
+    (date "2023-07-31")
+    (rev "V2.0")
+  )
   (junction (at 166.37 97.79) (diameter 0) (color 0 0 0 0)
   )
