File: electronics-v2/flight-controller-v2/sensors.kicad_sch (KiCad schematic)
At the start: 23 parts, among them J12 Conn_02x03_Odd_Even, U10 HMC5883L, U6 BMP280, U7 CS49E, U8 MPU-6050, U9 LM393

Commit message: fixes in routing
Parts:
- removed J12: Conn_02x03_Odd_Even, Connector_IDC:IDC-Header_2x03_P2.54mm_Vertical, symbol Connector_Generic:Conn_02x03_Odd_Even
Connections:
- net INT_I2C_SCL renamed SENSOR_I2C_SCL
- net INT_I2C_SDA renamed SENSOR_I2C_SDA
Other:
- note removed: "I2C address: 0x52"
- note removed: "TOF sensor"
Changed lines of the file:
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@@
-    (stroke (width 0) (type default) (color 0 0 0 0))
-  )
-  (polyline (pts (xy 92.71 80.01) (xy 92.71 25.4))
     (stroke (width 0) (type default) (color 0 0 0 0))
   )
@@
     (stroke (width 0) (type default) (color 0 0 0 0))
   )
-  (polyline (pts (xy 45.72 80.01) (xy 92.71 80.01))
-    (stroke (width 0) (type default) (color 0 0 0 0))
-  )
   (wire (pts (xy 209.55 111.76) (xy 209.55 110.49))
     (stroke (width 0) (type default) (color 0 0 0 0))
@@
     (stroke (width 0) (type default) (color 0 0 0 0))
   )
-  (polyline (pts (xy 45.72 25.4) (xy 45.72 80.01))
-    (stroke (width 0) (type default) (color 0 0 0 0))
-  )
   (polyline (pts (xy 92.71 86.36) (xy 92.71 151.13))
     (stroke (width 0) (type default) (color 0 0 0 0))
@@
   )
   (wire (pts (xy 167.64 129.54) (xy 167.64 134.62))
-    (stroke (width 0) (type default) (color 0 0 0 0))
-  )
-  (polyline (pts (xy 45.72 25.4) (xy 92.71 25.4))
     (stroke (width 0) (type default) (color 0 0 0 0))
   )
@@
     (effects (font (size 2.54 2.54) (thickness 0.508) bold) (justify right bottom))
   )
-  (text "TOF sensor" (at 80.01 33.02 180)
-    (effects (font (size 2.54 2.54) (thickness 0.508) bold) (justify right bottom))
-  )
-  (text "I2C address:\n0x1E" (at 186.69 116.84 0)
+  (text "I2C address:\n0x1E" (at 185.42 135.89 0)
     (effects (font (size 1.27 1.27) (thickness 0.254) bold) (justify left bottom))
   )
@@
     (effects (font (size 2.54 2.54) (thickness 0.508) bold) (justify right bottom))
   )
-  (text "I2C address:\n0x52" (at 64.77 67.31 0)
-    (effects (font (size 1.27 1.27) (thickness 0.254) bold) (justify left bottom))
-  )
   (label "IMU_VDD" (at 138.43 97.79 0)
     (effects (font (size 1.27 1.27)) (justify left bottom))
@@
     (effects (font (size 1.27 1.27)) (justify left bottom))
   )
-  (hierarchical_label "INT_I2C_SDA" (shape bidirectional) (at 199.39 125.73 180)
+  (hierarchical_label "SENSOR_I2C_SDA" (shape bidirectional) (at 199.39 125.73 180)
     (effects (font (size 1.27 1.27)) (justify right))
   )
-  (hierarchical_label "VLX_SCL" (shape bidirectional) (at 76.2 57.15 0)
-    (effects (font (size 1.27 1.27)) (justify left))
-  )
-  (hierarchical_label "INT_I2C_SDA" (shape bidirectional) (at 116.84 116.84 180)
+  (hierarchical_label "SENSOR_I2C_SDA" (shape bidirectional) (at 116.84 116.84 180)
     (effects (font (size 1.27 1.27)) (justify right))
   )
@@
     (effects (font (size 1.27 1.27)) (justify right))
   )
-  (hierarchical_label "VLX_XSHUT" (shape input) (at 63.5 54.61 180)
+  (hierarchical_label "SENSOR_I2C_SCL" (shape bidirectional) (at 199.39 123.19 180)
     (effects (font (size 1.27 1.27)) (justify right))
   )
-  (hierarchical_label "INT_I2C_SCL" (shape bidirectional) (at 199.39 123.19 180)
+  (hierarchical_label "SENSOR_I2C_SDA" (shape bidirectional) (at 64.77 129.54 180)
     (effects (font (size 1.27 1.27)) (justify right))
   )
-  (hierarchical_label "VLX_INT" (shape output) (at 76.2 54.61 0)
-    (effects (font (size 1.27 1.27)) (justify left))
-  )
-  (hierarchical_label "VLX_SDA" (shape bidirectional) (at 63.5 57.15 180)
+  (hierarchical_label "SENSOR_I2C_SCL" (shape bidirectional) (at 64.77 127 180)
     (effects (font (size 1.27 1.27)) (justify right))
   )
-  (hierarchical_label "INT_I2C_SDA" (shape bidirectional) (at 64.77 129.54 180)
+  (hierarchical_label "SENSOR_I2C_SCL" (shape bidirectional) (at 116.84 119.38 180)
     (effects (font (size 1.27 1.27)) (justify right))
   )
-  (hierarchical_label "INT_I2C_SCL" (shape bidirectional) (at 64.77 127 180)
-    (effects (font (size 1.27 1.27)) (justify right))
-  )
-  (hierarchical_label "INT_I2C_SCL" (shape bidirectional) (at 116.84 119.38 180)
-    (effects (font (size 1.27 1.27)) (justify right))
-  )
   (symbol (lib_id "power:GND") (at 64.77 118.11 0) (unit 1)
     (in_bom yes) (on_board yes) (fields_autoplaced)
-    (property "Reference" "#PWR075" (id 0) (at 64.77 124.46 0)
+    (property "Reference" "#PWR076" (id 0) (at 64.77 124.46 0)
       (effects (font (size 1.27 1.27)) hide)
     )
@@
     )
     (property "Datasheet" "" (id 3) (at 152.4 106.68 0)
-      (effects (font (size 1.27 1.27)) hide)
-    )
-    (pin "1")
-  )
-  (symbol (lib_id "power:GND") (at 63.5 59.69 270) (unit 1)
-    (in_bom yes) (on_board yes)
-    (property "Reference" "#PWR073" (id 0) (at 57.15 59.69 0)
-      (effects (font (size 1.27 1.27)) hide)
-    )
-    (property "Value" "GND" (id 1) (at 59.69 59.69 90)
-      (effects (font (size 1.27 1.27)) (justify right))
-    )
-    (property "Footprint" "" (id 2) (at 63.5 59.69 0)
-      (effects (font (size 1.27 1.27)) hide)
-    )
-    (property "Datasheet" "" (id 3) (at 63.5 59.69 0)
       (effects (font (size 1.27 1.27)) hide)
     )
@@
   (symbol (lib_id "power:+3.3V") (at 64.77 107.95 0) (unit 1)
     (in_bom yes) (on_board yes) (fields_autoplaced)
-    (property "Reference" "#PWR074" (id 0) (at 64.77 111.76 0)
+    (property "Reference" "#PWR075" (id 0) (at 64.77 111.76 0)
       (effects (font (size 1.27 1.27)) hide)
     )
@@
     (pin "1")
   )
-  (symbol (lib_id "Connector_Generic:Conn_02x03_Odd_Even") (at 68.58 57.15 0) (unit 1)
-    (in_bom yes) (on_board yes) (fields_autoplaced)
-    (property "Reference" "J12" (id 0) (at 69.85 48.26 0))
-    (property "Value" "Conn_02x03_Odd_Even" (id 1) (at 69.85 50.8 0))
-    (property "Footprint" "Connector_IDC:IDC-Header_2x03_P2.54mm_Vertical" (id 2) (at 68.58 57.15 0)
-      (effects (font (size 1.27 1.27)) hide)
-    )
-    (property "Datasheet" "~" (id 3) (at 68.58 57.15 0)
-      (effects (font (size 1.27 1.27)) hide)
-    )
-    (pin "1")
-    (pin "2")
-    (pin "3")
-    (pin "4")
-    (pin "5")
-    (pin "6")
-  )
-  (symbol (lib_id "power:+3.3V") (at 76.2 59.69 270) (unit 1)
-    (in_bom yes) (on_board yes)
-    (property "Reference" "#PWR077" (id 0) (at 72.39 59.69 0)
-      (effects (font (size 1.27 1.27)) hide)
-    )
-    (property "Value" "+3.3V" (id 1) (at 85.09 59.69 90)
-      (effects (font (size 1.27 1.27)) (justify right))
-    )
-    (property "Footprint" "" (id 2) (at 76.2 59.69 0)
-      (effects (font (size 1.27 1.27)) hide)
-    )
-    (property "Datasheet" "" (id 3) (at 76.2 59.69 0)
-      (effects (font (size 1.27 1.27)) hide)
-    )
-    (pin "1")
-  )
   (symbol (lib_id "power:GND") (at 82.55 118.11 0) (unit 1)
     (in_bom yes) (on_board yes) (fields_autoplaced)
@@
   (symbol (lib_id "power:+3.3V") (at 55.88 138.43 0) (unit 1)
     (in_bom yes) (on_board yes) (fields_autoplaced)
-    (property "Reference" "#PWR072" (id 0) (at 55.88 142.24 0)
+    (property "Reference" "#PWR074" (id 0) (at 55.88 142.24 0)
       (effects (font (size 1.27 1.27)) hide)
     )
@@
   )
   (symbol (lib_id "Sensor_Motion:MPU-6050") (at 134.62 124.46 0) (unit 1)
-    (in_bom yes) (on_board yes) (fields_autoplaced)
-    (property "Reference" "U8" (id 0) (at 136.6394 140.97 0)
-      (effects (font (size 1.27 1.27)) (justify left))
-    )
-    (property "Value" "MPU-6050" (id 1) (at 136.6394 143.51 0)
+    (in_bom yes) (on_board yes)
+    (property "Reference" "U8" (id 0) (at 142.24 106.68 0)
+      (effects (font (size 1.27 1.27)) (justify left))
+    )
+    (property "Value" "MPU-6050" (id 1) (at 138.43 109.22 0)
       (effects (font (size 1.27 1.27)) (justify left))
     )
@@
   (symbol (lib_id "power:GND") (at 74.93 142.24 0) (unit 1)
     (in_bom yes) (on_board yes) (fields_autoplaced)
-    (property "Reference" "#PWR076" (id 0) (at 74.93 148.59 0)
-      (effects (font (size 1.27 1.27)) hide)
-    )
+    (property "Reference" "#PWR077" (id 0) (at 74.93 148.59 0)
+      (effects (font (size 1.27 1.27)) hide)
+    )

Commit message: generate schematic
Other:
- title: (none) -> UAV TVC Goose Flight Controller
Changed lines of the file:
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@@
 (kicad_sch (version 20211123) (generator eeschema)
   (paper "A4")
+  (title_block
+    (title "UAV TVC Goose Flight Controller")
+    (date "2023-07-31")
+    (rev "V2.0")
+  )
   (junction (at 212.09 110.49) (diameter 0) (color 0 0 0 0)
   )

Commit message: fix Vref in Hall comeprator, update schematic, add moving average to vel
Parts:
- R30: value 100k -> 200k
- R31: value 100k -> 220k
Other:
- note added: "histeresis: Vref = 1.728V R33/R32 = 66.667 Vth = 1.75V Vtl = 1.70V"
Changed lines of the file:
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@@
     (effects (font (size 2.54 2.54) (thickness 0.508) bold) (justify right bottom))
+  )
+  (text "histeresis:\nVref = 1.728V\nR33/R32 = 66.667\n\nVth = 1.75V\nVtl = 1.70V"
+    (at 132.08 67.31 0)
+    (effects (font (size 1.27 1.27)) (justify left bottom))
   )
   (text "I2C address:\n0x1E" (at 185.42 135.89 0)
@@
       (effects (font (size 1.27 1.27)) (justify left))
     )
-    (property "Value" "100k" (id 1) (at 160.02 58.4199 0)
+    (property "Value" "200k" (id 1) (at 160.02 58.4199 0)
       (effects (font (size 1.27 1.27)) (justify left))
     )
@@
       (effects (font (size 1.27 1.27)) (justify left))
     )
-    (property "Value" "100k" (id 1) (at 160.02 68.5799 0)
-      (effects (font (size 1.27 1.27)) (justify left))
-    )
+    (property "Value" "220k" (id 1) (at 160.02 68.5799 0)
+      (effects (font (size 1.27 1.27)) (justify left))
+    )
