File: hardware/auxiliary-modules/auxiliary-modules.kicad_sch (KiCad schematic)
At the start: 37 parts, among them J1 IDC-10, J2 Conn_01x07, J3 IDC-10, J4 Conn_01x04, J5 IDC-10, U1 NTS0102, U2 CS49E, U3 LM393, U4 NTS0102

Commit message: aux clean footprints
Parts:
- added H1, H2, H3: MountingHole_Pad, MountingHole:MountingHole_3.5mm_Pad_Via, symbol Mechanical:MountingHole_Pad
- D1: renamed from D2; footprint (none) -> LED_SMD:LED_0603_1608Metric
- J1: renamed from J5; footprint goose:IDC-10-horizontal -> auxiliary:IDC-10_vertical
- J2: renamed from J1; footprint goose:IDC-10-horizontal -> auxiliary:IDC-10_vertical
- J3: renamed from J4; footprint (none) -> auxiliary:header_1x4
- J4: renamed from J3; footprint goose:IDC-10-horizontal -> auxiliary:IDC-10_vertical
- J5: renamed from J2; footprint (none) -> auxiliary:header_1x7
- R1: renamed from R2; footprint (none) -> Resistor_SMD:R_0603_1608Metric
- R2: renamed from R7; footprint (none) -> Resistor_SMD:R_0603_1608Metric
- R3: renamed from R5; footprint (none) -> Resistor_SMD:R_0603_1608Metric
- R4: renamed from R1; footprint (none) -> Resistor_SMD:R_0603_1608Metric
- R5: renamed from R6; footprint (none) -> Resistor_SMD:R_0603_1608Metric
- U1: renamed from U2; footprint (none) -> auxiliary:hall
- U2: renamed from U4; footprint (none) -> auxiliary:NTS0102
- U3: footprint (none) -> auxiliary:LM393
- U4: renamed from U1; footprint (none) -> auxiliary:NTS0102
- renumbered C8 to C1, C3 to C10, C4 to C11, C15 to C12, C5 to C13, C6 to C14, C14 to C15, C11 to C2, C7 to C3, C9 to C4, C10 to C5, C12 to C6, C1 to C7, C2 to C8, C13 to C9, L4 to L1, L5 to L2, L1 to L3, L2 to L4, L3 to L5
Connections:
- net FLOW_GND: now also H2.1
- net RANGE_GND: now also H3.1
- net TACH_GND: now also H1.1
Other:
- moved on the sheet: C10, C11, C12, J2, J5, L4

Commit message: ready?
Parts:
- removed RV1: 100k, symbol Device:R_Potentiometer
- removed RV2: 10k, symbol Device:R_Potentiometer
- renumbered C13 to C10, C14 to C11, C15 to C12, C10 to C13, C11 to C14, C12 to C15, J5 to J2, J2 to J5, L5 to L4, L4 to L5
Connections:
- no-connect marks 15 -> 14
Changed lines of the file:
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@@
 	)
 	(no_connect
-		(at 158.75 74.93)
-	)
-	(no_connect
 		(at 176.53 148.59)
 	)
@@
 	(wire
 		(pts
-			(xy 139.7 80.01) (xy 140.97 80.01)
-		)
-		(stroke
-			(width 0)
-			(type default)
-		)
-	)
-	(wire
-		(pts
 			(xy 194.31 48.26) (xy 193.04 48.26)
 		)
@@
 	(wire
 		(pts
-			(xy 139.7 78.74) (xy 139.7 80.01)
-		)
-		(stroke
-			(width 0)
-			(type default)
-		)
-	)
-	(wire
-		(pts
 			(xy 91.44 142.24) (xy 91.44 143.51)
 		)
@@
 	(wire
 		(pts
-			(xy 139.7 69.85) (xy 140.97 69.85)
-		)
-		(stroke
-			(width 0)
-			(type default)
-		)
-	)
-	(wire
-		(pts
 			(xy 44.45 62.23) (xy 54.61 62.23)
 		)
@@
 	(wire
 		(pts
-			(xy 139.7 71.12) (xy 139.7 69.85)
-		)
-		(stroke
-			(width 0)
-			(type default)
-		)
-	)
-	(wire
-		(pts
 			(xy 68.58 45.72) (xy 68.58 46.99)
 		)
@@
 		)
 	)
-	(global_label "TACH_5V"
-		(shape input)
-		(at 140.97 69.85 0)
-		(fields_autoplaced yes)
-		(effects
-			(font
-				(size 1.27 1.27)
-			)
-			(justify left)
-		)
-		(property "Intersheetrefs" "${INTERSHEET_REFS}"
-			(at 151.8776 69.85 0)
-			(effects
-				(font
-					(size 1.27 1.27)
-				)
-				(justify left)
-				(hide yes)
-			)
-		)
-	)
 	(global_label "FLOW_MOSI"
 		(shape input)
@@
 		)
 	)
-	(global_label "TACH_GND"
-		(shape input)
-		(at 140.97 80.01 0)
-		(fields_autoplaced yes)
-		(effects
-			(font
-				(size 1.27 1.27)
-			)
-			(justify left)
-		)
-		(property "Intersheetrefs" "${INTERSHEET_REFS}"
-			(at 153.45 80.01 0)
-			(effects
-				(font
-					(size 1.27 1.27)
-				)
-				(justify left)
-				(hide yes)
-			)
-		)
-	)
 	(global_label "FLOW_3.3V"
 		(shape input)
@@
 		(on_board yes)
 		(dnp no)
-		(property "Reference" "C10"
+		(property "Reference" "C13"
 			(at 208.28 147.3199 0)
 			(effects
@@
 			(project "auxiliary-modules"
 				(path "/90296362-2817-4339-8dfe-87b7e4356586"
-					(reference "C10")
+					(reference "C13")
 					(unit 1)
 				)
@@
 		(on_board yes)
 		(dnp no)
-		(property "Reference" "C14"
+		(property "Reference" "C11"
 			(at 83.82 146.0499 0)
 			(effects
@@
 			(project "auxiliary-modules"
 				(path "/90296362-2817-4339-8dfe-87b7e4356586"
-					(reference "C14")
+					(reference "C11")
 					(unit 1)
 				)
@@
 	)
 	(symbol
-		(lib_id "Device:R_Potentiometer")
-		(at 139.7 74.93 0)
-		(unit 1)
-		(exclude_from_sim no)
-		(in_bom yes)
-		(on_board yes)
-		(dnp no)
-		(fields_autoplaced yes)
-		(property "Reference" "RV1"
-			(at 137.16 73.6599 0)
-			(effects
-				(font
-					(size 1.27 1.27)
-				)
-				(justify right)
-			)
-		)
-		(property "Value" "100k"
-			(at 137.16 76.1999 0)
-			(effects
-				(font
-					(size 1.27 1.27)
-				)
-				(justify right)
-			)
-		)
-		(property "Footprint" ""
-			(at 139.7 74.93 0)
-			(effects
-				(font
-					(size 1.27 1.27)
-				)
-				(hide yes)
-			)
-		)
-		(property "Datasheet" "~"
-			(at 139.7 74.93 0)
-			(effects
-				(font
-					(size 1.27 1.27)
-				)
-				(hide yes)
-			)
-		)
-		(property "Description" "Potentiometer"
-			(at 139.7 74.93 0)
-			(effects
-				(font
-					(size 1.27 1.27)
-				)
-				(hide yes)
-			)
-		)
-		(pin "1"
-		)
-		(pin "3"
-		)
-		(pin "2"
-		)
-		(instances
-			(project ""
-				(path "/90296362-2817-4339-8dfe-87b7e4356586"
-					(reference "RV1")
-					(unit 1)
-				)
-			)
-		)
-	)
-	(symbol
 		(lib_id "Device:L")
 		(at 74.93 142.24 270)
@@
 		(dnp no)
 		(fields_autoplaced yes)
-		(property "Reference" "L5"
+		(property "Reference" "L4"
 			(at 74.93 137.16 90)
 			(effects
@@
 			(project "auxiliary-modules"
 				(path "/90296362-2817-4339-8dfe-87b7e4356586"
-					(reference "L5")
-					(unit 1)
-				)
-			)
-		)
-	)
-	(symbol
-		(lib_id "Device:R_Potentiometer")
-		(at 162.56 74.93 270)
-		(mirror x)
-		(unit 1)
-		(exclude_from_sim no)
-		(in_bom yes)
-		(on_board yes)
-		(dnp no)
-		(property "Reference" "RV2"
-			(at 162.56 78.74 90)
-			(effects
-				(font
-					(size 1.27 1.27)
-				)
-			)
-		)
-		(property "Value" "10k"
-			(at 162.56 81.28 90)
-			(effects
-				(font
-					(size 1.27 1.27)
-				)
-			)
-		)
-		(property "Footprint" ""
-			(at 162.56 74.93 0)
-			(effects
-				(font
-					(size 1.27 1.27)
-				)
-				(hide yes)
-			)
-		)
-		(property "Datasheet" "~"
-			(at 162.56 74.93 0)
-			(effects
-				(font
-					(size 1.27 1.27)
-				)
-				(hide yes)
-			)
-		)
-		(property "Description" "Potentiometer"
-			(at 162.56 74.93 0)
-			(effects
-				(font
-					(size 1.27 1.27)
-				)
-				(hide yes)
-			)
-		)
-		(pin "1"
-		)
-		(pin "3"
-		)
-		(pin "2"
-		)
-		(instances
-			(project "auxiliary-modules"
-				(path "/90296362-2817-4339-8dfe-87b7e4356586"
-					(reference "RV2")
+					(reference "L4")
 					(unit 1)
 				)
@@
 		(on_board yes)
 		(dnp no)
-		(property "Reference" "C12"
+		(property "Reference" "C15"
 			(at 237.49 147.3199 0)
 			(effects
@@
 			(project "auxiliary-modules"
 				(path "/90296362-2817-4339-8dfe-87b7e4356586"
-					(reference "C12")
+					(reference "C15")
 					(unit 1)
 				)
@@
 		(on_board yes)
 		(dnp no)
-		(property "Reference" "C13"
+		(property "Reference" "C10"
 			(at 66.04 146.0499 0)
 			(effects
@@
 			(project "auxiliary-modules"
 				(path "/90296362-2817-4339-8dfe-87b7e4356586"
-					(reference "C13")
+					(reference "C10")
 					(unit 1)
 				)
@@
 		(dnp no)
 		(fields_autoplaced yes)
-		(property "Reference" "L4"
+		(property "Reference" "L5"
 			(at 217.17 138.43 90)
 			(effects
@@
 			(project "auxiliary-modules"
 				(path "/90296362-2817-4339-8dfe-87b7e4356586"
-					(reference "L4")
+					(reference "L5")
 					(unit 1)
 				)
@@
 		(dnp no)
 		(fields_autoplaced yes)
-		(property "Reference" "J2"
+		(property "Reference" "J5"
 			(at 182.88 134.62 0)
 			(effects
@@
 			(project "auxiliary-modules"
 				(path "/90296362-2817-4339-8dfe-87b7e4356586"
-					(reference "J2")
+					(reference "J5")
 					(unit 1)
 				)
@@
 		(dnp no)
 		(fields_autoplaced yes)
-		(property "Reference" "J5"
+		(property "Reference" "J2"
 			(at 242.57 120.6499 0)
 			(effects
@@
 			(project ""
 				(path "/90296362-2817-4339-8dfe-87b7e4356586"
-					(reference "J5")
+					(reference "J2")
 					(unit 1)
 				)
@@
 		(on_board yes)
 		(dnp no)
-		(property "Reference" "C15"
+		(property "Reference" "C12"
 			(at 95.25 146.0499 0)
 			(effects
@@
 			(project "auxiliary-modules"
 				(path "/90296362-2817-4339-8dfe-87b7e4356586"
-					(reference "C15")
+					(reference "C12")
 					(unit 1)
 				)
@@
 		(on_board yes)
 		(dnp no)
-		(property "Reference" "C11"
+		(property "Reference" "C14"
 			(at 226.06 147.3199 0)
 			(effects
@@
 			(project "auxiliary-modules"
 				(path "/90296362-2817-4339-8dfe-87b7e4356586"
-					(reference "C11")
+					(reference "C14")
 					(unit 1)
 				)
