File: hardware/flight-controller/sensors.kicad_sch (KiCad schematic)
At the start: 0 parts

Commit message: sensors, power, actuators, filters
Parts:
- added C38, C39, C40, C41, C42, C43, C46: 100n, symbol Device:C
- added C44: 220n, symbol Device:C
- added C45: 4u7, symbol Device:C
- added C47: 2n2, symbol Device:C
- added D6: LED, symbol Device:LED
- added R29, R30: 100k, symbol Device:R
- added R31: 1k, symbol Device:R
- added R32: 200k, symbol Device:R
- added R33: 1k5, symbol Device:R
- added R34: 220k, symbol Device:R
- added U10: MPU-6050, Sensor_Motion:InvenSense_QFN-24_4x4mm_P0.5mm, symbol Sensor_Motion:MPU-6050
- added U6: CS49E, symbol Connector_Generic:Conn_01x03
- added U7: LM393, symbol Comparator:LM393
- added U8: HMC5883L, symbol goose:HMC5883L
- added U9: BMP280, Package_LGA:Bosch_LGA-8_2x2.5mm_P0.65mm_ClockwisePinNumbering, symbol Sensor_Pressure:BMP280
Connections:
- new net: D6.1 (K), R31.1
- new net +3.3V: C38.1, C39.1, C40.1, C41.1, C42.1, C43.1, D6.2 (A), R30.1, R32.1, U10.13 (VDD), U10.8 (VLOGIC), U6.1 (Pin_1), U7.8 (V+), U8.13 (VDDIO), U8.2 (VDD), U8.4 (S1), U9.2 (CSB), U9.5 (SDO), U9.6 (VDDIO), U9.8 (VDD)
- new net BAR_SCL: U9.4 (SCK)
- new net BAR_SDA: U9.3 (SDI)
- new net GND: C38.2, C39.2, C40.2, C41.2, C42.2, C43.2, C45.2, C46.2, C47.2, R34.2, U10.1 (CLKIN), U10.11 (FSYNC), U10.18 (GND), U10.9 (AD0), U6.2 (Pin_2), U7.4 (V-), U8.11 (GND), U8.9 (GND), U9.1 (GND), U9.7 (GND)
- new net HALL: R29.2, R30.2, R31.2, R33.1, U6.3 (Pin_3), U7.1
- new net HALL_FB: R29.1, R33.2, U7.3 (+)
- new net HALL_REF: R32.2, R34.1, U7.2 (-)
- new net IMU_CPOUT: C47.1, U10.20 (CPOUT)
- new net IMU_INT: U10.12 (INT)
- new net IMU_REGOUT: C46.1, U10.10 (REGOUT)
- new net IMU_SCL: U10.23 (SCL)
- new net IMU_SDA: U10.24 (SDA)
- new net MAG_C1: C45.1, U8.10 (C1)
- new net MAG_INT: U8.15 (DRDY)
- new net MAG_SCL: U8.1 (SCL)
- new net MAG_SDA: U8.16 (SDA)
- new net MAG_SETC: C44.2, U8.12 (SETC)
- new net MAG_SETP: C44.1, U8.8 (SETP)
- no-connect marks 0 -> 2
Other:
- note added: "I2C address: 0x1E (7-bit)"
- note added: "I2C address: 0x68 (7-bit)"
- note added: "I2C address: 0x77 (7-bit)"
- note added: "IMU"
- note added: "barometer"
- note added: "magnetometer"
- note added: "rotor velocity measurement"

Commit message: schematic cleanup
Parts:
- added C14, C15, C17, C18, C3, C4, C48, C49, C5, C50, C51, C58, C59, C6: 4u7, symbol Device:C
- added C52, C53: 100n, symbol Device:C
- added J11, J13, J15: IDC-10, symbol Connector_Generic:Conn_02x05_Odd_Even
- added J14: IDC-6, symbol Connector_Generic:Conn_02x03_Odd_Even
- added L1, L10, L14, L2, L4, L5, L9: 2u2, symbol Device:L
- added R36, R37: 10, symbol Device:R
- added R38: 4k7, symbol Device:R
- added U11: INA226, Package_SO:VSSOP-10_3x3mm_P0.5mm, symbol Sensor_Energy:INA226
Connections:
- net +3.3V: now also C18.1, C48.1, C53.1, C58.1, C6.1, L14.1, L2.1, L5.1, L9.1, R38.1, U11.6 (VS)
- net GND: now also C14.2, C15.2, C17.2, C18.2, C3.2, C4.2, C48.2, C49.2, C5.2, C50.2, C51.2, C53.2, C58.2, C59.2, C6.2, J11.10 (Pin_10), J13.10 (Pin_10), J14.6 (Pin_6), J15.10 (Pin_10), U11.1 (A1), U11.2 (A0), U11.7 (GND)
- net BAR_SCL renamed SCL
- net SCL: now also U11.5 (SCL)
- net BAR_SDA renamed SDA
- net SDA: now also U11.4 (SDA)
- net HALL renamed HALL_OUT
- new net: C52.1, R36.2, U11.10 (Vin+)
- new net: C52.2, R37.2, U11.8 (Vbus), U11.9 (Vin-)
- new net +5V: C17.1, C49.1, C5.1, L1.1, L10.1, L4.1
- new net FLOW_3V3: C50.1, J11.4 (Pin_4), L9.2
- new net FLOW_5V: C51.1, J11.2 (Pin_2), L10.2
- new net FLOW_CS: J11.8 (Pin_8)
- new net FLOW_INT: J11.6 (Pin_6)
- new net FLOW_MISO: J11.1 (Pin_1)
- new net FLOW_MOSI: J11.3 (Pin_3)
- new net FLOW_SCK: J11.5 (Pin_5)
- new net GPS_3V3: C59.1, J14.1 (Pin_1), L14.2
- new net GPS_RX: J14.5 (Pin_5)
- new net GPS_TX: J14.3 (Pin_3)
- new net HALL_3V3: C15.1, J15.4 (Pin_4), L5.2
- new net HALL_5V: C14.1, J15.2 (Pin_2), L4.2
- new net HALL_VEL: J15.6 (Pin_6)
- new net PWR_INT: R38.2, U11.3 (~{Alert})
- new net RANGE_3V3: C4.1, J13.4 (Pin_4), L2.2
- new net RANGE_5V: C3.1, J13.2 (Pin_2), L1.2
- new net RANGE_ECHO: J13.6 (Pin_6)
- new net RANGE_TRIG: J13.8 (Pin_8)
- new net SHUNT_HIGH: R36.1
- new net SHUNT_LOW: R37.1
- no-connect marks 2 -> 17
Other:
- note added: "I2C address: 0x40 (7-bit)"
- note added: "accelerometer & gyroscope"
- note added: "external gps"
- note added: "external motor velocity"
- note added: "external optical flow"
- note added: "external rangefinder"
- note added: "power monitor"
- note added: "to HC-SR04 adapter board"
- note added: "to Hall & opamp near rotor magnets"
- note added: "to PMW3901 adapter board"
- note added: "to UBX-G7020"
- note removed: "IMU"
- moved on the sheet: C38, C39, C40, C41, C42, C43, C44, C45, C46, C47, D6, R29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

Commit message: still working
Parts:
- removed C14, C15, C17, C18, C3, C4, C48, C49, C5, C50, C51, C58, C59, C6: 4u7, symbol Device:C
- removed C42, C52, C53: 100n, symbol Device:C
- removed D6: LED, symbol Device:LED
- removed J11, J13, J15: IDC-10, symbol Connector_Generic:Conn_02x05_Odd_Even
- removed J14: IDC-6, symbol Connector_Generic:Conn_02x03_Odd_Even
- removed L1, L10, L14, L2, L4, L5, L9: 2u2, symbol Device:L
- removed R31: 1k, symbol Device:R
- removed R32: 200k, symbol Device:R
- removed R33: 1k5, symbol Device:R
- removed R34: 220k, symbol Device:R
- removed R36, R37: 10, symbol Device:R
- removed R38: 4k7, symbol Device:R
- removed U11: INA226, Package_SO:VSSOP-10_3x3mm_P0.5mm, symbol Sensor_Energy:INA226
- removed U6: CS49E, symbol Connector_Generic:Conn_01x03
- removed U7: LM393, symbol Comparator:LM393
- added C27, C34, C35, C37: 100n, Capacitor_SMD:C_0603_1608Metric, symbol Device:C
- added C33, C36: 10u, symbol Device:C
- added Q2: S8550, Package_TO_SOT_SMD:SOT-23, symbol Device:Q_PNP_BEC
- added R23, R24, R25, R26: 4k7, Resistor_SMD:R_0603_1608Metric, symbol Device:R
- added R27: 20k, Resistor_SMD:R_0603_1608Metric, symbol Device:R
- added R28: 8k2, Resistor_SMD:R_0603_1608Metric, symbol Device:R
- added U9: HX711, Package_SO:SOP-16_3.9x9.9mm_P1.27mm, symbol Analog_ADC:HX711
- C24: renamed from C41; footprint (none) -> Capacitor_SMD:C_0603_1608Metric
- C25: renamed from C39; footprint (none) -> Capacitor_SMD:C_0603_1608Metric
- C26: renamed from C40; footprint (none) -> Capacitor_SMD:C_0603_1608Metric
- C28: renamed from C43; footprint (none) -> Capacitor_SMD:C_0603_1608Metric
- C29: renamed from C44; footprint (none) -> Capacitor_SMD:C_0603_1608Metric
- C31: renamed from C46; footprint (none) -> Capacitor_SMD:C_0603_1608Metric
- C32: renamed from C47; footprint (none) -> Capacitor_SMD:C_0603_1608Metric
- C38: footprint (none) -> Capacitor_SMD:C_0603_1608Metric
- R29, R30: value 100k -> 100; footprint (none) -> Resistor_SMD:R_0603_1608Metric
- renumbered C45 to C30, U8 to U6, U10 to U7, U9 to U8
Connections:
- net +3.3V: now also C27.1, C33.1, C34.1, Q2.2 (E), R23.1, R24.1, R25.1, R26.1, U9.1 (VSUP), U9.16 (DVDD); no longer C38.1, R30.1
- net GND: now also C27.2, C33.2, C34.2, C35.2, C36.2, R28.2, U9.10 (INB+), U9.14 (XI), U9.5 (AGND), U9.9 (INB-)
- net IMU_SCL: now also R24.2
- net IMU_SDA: now also R23.2
- net MAG_SCL: now also R26.2
- net MAG_SDA: now also R25.2
- net HALL_FB renamed LOAD_SP
- net HALL_OUT: no longer names the net of R29.2
- net HALL_OUT: now also C37.1, U9.8 (INA+); no longer R30.2
- net SCL renamed MISC_SCL
- net SDA renamed MISC_SDA
- new net: R27.2, R28.1, U9.4 (VFB)
- new net: C38.1, U9.6 (VBG)
- new net: Q2.1 (B), U9.2 (BASE)
- new net: C37.2, R30.1, U9.7 (INA-)
- new net LOAD_DOUT: U9.12 (DOUT)
- new net LOAD_EP: C35.1, C36.1, Q2.3 (C), R27.1, U9.3 (AVDD)
- new net LOAD_RATE: U9.15 (RATE)
- new net LOAD_SCK: U9.11 (PD_SCK)
- new net LOAD_SN: R30.2
- no-connect marks 17 -> 3
Other:
- note added: "RATE: 0 -> 10Hz 1 -> 80Hz"
- note added: "load cell ADC"
- note removed: "I2C address: 0x40 (7-bit)"
- note removed: "external gps"
- note removed: "external motor velocity"
- note removed: "external optical flow"
- note removed: "external rangefinder"
- note removed: "power monitor"
- note removed: "rotor velocity measurement"
- note removed: "to HC-SR04 adapter board"
- note removed: "to Hall & opamp near rotor magnets"
- note removed: "to PMW3901 adapter board"
- note removed: "to UBX-G7020"
- moved on the sheet: C24, C25, C26, C28, C29, C30, C31, C32, U6, U7, U8

Commit message: clean footprints
Parts:
- U6: footprint (none) -> goose:HMC5883L_handsolder
- U7: footprint Sensor_Motion:InvenSense_QFN-24_4x4mm_P0.5mm -> goose:MPU6050_handsolder
- U8: footprint Package_LGA:Bosch_LGA-8_2x2.5mm_P0.65mm_ClockwisePinNumbering -> goose:BMP280_handsolder
- U9: footprint Package_SO:SOP-16_3.9x9.9mm_P1.27mm -> goose:hx711
Changed lines of the file:
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@@
 			)
 		)
-		(property "Footprint" "Package_LGA:Bosch_LGA-8_2x2.5mm_P0.65mm_ClockwisePinNumbering"
+		(property "Footprint" "goose:BMP280_handsolder"
 			(at 245.11 81.28 0)
 			(effects
@@
 			)
 		)
-		(property "Footprint" "Sensor_Motion:InvenSense_QFN-24_4x4mm_P0.5mm"
+		(property "Footprint" "goose:MPU6050_handsolder"
 			(at 64.77 81.28 0)
 			(effects
@@
 			)
 		)
-		(property "Footprint" ""
+		(property "Footprint" "goose:HMC5883L_handsolder"
 			(at 170.18 41.148 0)
 			(effects
@@
 			)
 		)
-		(property "Datasheet" ""
+		(property "Datasheet" "https://www.farnell.com/datasheets/1683374.pdf"
 			(at 170.18 41.148 0)
 			(effects
@@
 			)
 		)
-		(property "Footprint" "Package_SO:SOP-16_3.9x9.9mm_P1.27mm"
+		(property "Footprint" "goose:hx711"
 			(at 121.92 137.16 0)
 			(effects

Commit message: clean footprints
Parts:
- C30, C33, C36: footprint (none) -> Capacitor_SMD:C_0603_1608Metric
- Q2: footprint Package_TO_SOT_SMD:SOT-23 -> goose:SOT-23
- U9: footprint goose:hx711 -> goose:HX711
Changed lines of the file:
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@@
 	(wire
 		(pts
-			(xy 43.18 132.08) (xy 45.72 132.08)
-		)
-		(stroke
-			(width 0)
-			(type default)
-		)
-	)
-	(wire
-		(pts
 			(xy 83.82 34.29) (xy 90.17 34.29)
 		)
@@
 	(wire
 		(pts
-			(xy 45.72 132.08) (xy 45.72 137.16)
-		)
-		(stroke
-			(width 0)
-			(type default)
-		)
-	)
-	(wire
-		(pts
 			(xy 237.49 39.37) (xy 245.11 39.37)
 		)
@@
 		)
 	)
-	(global_label "LOAD_EN"
-		(shape input)
-		(at 43.18 132.08 180)
-		(fields_autoplaced yes)
-		(effects
-			(font
-				(size 1.27 1.27)
-			)
-			(justify right)
-		)
-		(property "Intersheetrefs" "${INTERSHEET_REFS}"
-			(at 32.0305 132.08 0)
-			(effects
-				(font
-					(size 1.27 1.27)
-				)
-				(justify right)
-				(hide yes)
-			)
-		)
-	)
 	(global_label "IMU_INT"
 		(shape input)
@@
 	(symbol
 		(lib_id "power:GND")
-		(at 45.72 137.16 0)
-		(unit 1)
-		(exclude_from_sim no)
-		(in_bom yes)
-		(on_board yes)
-		(dnp no)
-		(property "Reference" "#PWR077"
-			(at 45.72 143.51 0)
-			(effects
-				(font
-					(size 1.27 1.27)
-				)
-				(hide yes)
-			)
-		)
-		(property "Value" "GND"
-			(at 45.72 142.24 0)
-			(effects
-				(font
-					(size 1.27 1.27)
-				)
-			)
-		)
-		(property "Footprint" ""
-			(at 45.72 137.16 0)
-			(effects
-				(font
-					(size 1.27 1.27)
-				)
-				(hide yes)
-			)
-		)
-		(property "Datasheet" ""
-			(at 45.72 137.16 0)
-			(effects
-				(font
-					(size 1.27 1.27)
-				)
-				(hide yes)
-			)
-		)
-		(property "Description" "Power symbol creates a global label with name \"GND\" , ground"
-			(at 45.72 137.16 0)
-			(effects
-				(font
-					(size 1.27 1.27)
-				)
-				(hide yes)
-			)
-		)
-		(pin "1"
-		)
-		(instances
-			(project "flight-controller"
-				(path "/52d2474d-2865-43c6-846b-d5f8a367c5f4/422eb0b5-2ec1-41a7-81d9-981a304088f5"
-					(reference "#PWR077")
-					(unit 1)
-				)
-			)
-		)
-	)
-	(symbol
-		(lib_id "power:GND")
 		(at 143.51 114.3 0)
 		(unit 1)
@@
 			)
 		)
-		(property "Footprint" ""
+		(property "Footprint" "Capacitor_SMD:C_0603_1608Metric"
 			(at 65.7352 137.16 0)
 			(effects
@@
 			)
 		)
-		(property "Footprint" "goose:hx711"
+		(property "Footprint" "goose:HX711"
 			(at 121.92 137.16 0)
 			(effects
@@
 			)
 		)
-		(property "Footprint" ""
+		(property "Footprint" "Capacitor_SMD:C_0603_1608Metric"
 			(at 133.0452 76.2 0)
 			(effects
@@
 			)
 		)
-		(property "Footprint" "Package_TO_SOT_SMD:SOT-23"
+		(property "Footprint" "goose:SOT-23"
 			(at 76.2 124.46 0)
 			(effects
@@
 			)
 		)
-		(property "Footprint" ""
+		(property "Footprint" "Capacitor_SMD:C_0603_1608Metric"
 			(at 136.1948 114.3 0)
 			(effects

Commit message: clean models
Parts:
- C31: renamed from C30; value 4u7 -> 4.7u
- R22: renamed from R23; value 4k7 -> 4.7k
- R23: renamed from R24; value 4k7 -> 4.7k
- R24: renamed from R25; value 4k7 -> 4.7k
- R25: renamed from R26; value 4k7 -> 4.7k
- R27: renamed from R28; value 8k2 -> 8.2k
- renumbered C24 to C25, C25 to C26, C26 to C27, C27 to C28, C28 to C29, C29 to C30, C31 to C32, C32 to C33, C33 to C34, C34 to C35, C35 to C36, C36 to C37, C37 to C38, C38 to C39, R27 to R26, R29 to R28, R30 to R29
