File: hardware/flight-controller/sensors.kicad_sch (KiCad schematic)
At the start: 28 parts, among them Q2 S8550, U6 HMC5883L, U7 MPU-6050, U8 BMP280, U9 HX711

Commit message: generate schematic in pdf
Other:
- title: UAV TVC Goose Flight Controller -> UAV TVC Goose II: Flight Controller
Changed lines of the file:
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@@
 	(paper "A4")
 	(title_block
-		(title "UAV TVC Goose Flight Controller")
+		(title "UAV TVC Goose II: Flight Controller")
 		(date "2024-08-05")
 		(rev "V2.1")
