File: hardware/flight-controller/connectors.kicad_sch (KiCad schematic)
At the start: 40 parts, among them J10 IDC-10, J3 IDC-10, J4 Conn_01x03, J5 Conn_01x03, J6 Conn_01x03, J7 IDC-10, J8 XT-60, J9 Conn_01x03

Commit message: generate schematic in pdf
Other:
- title: UAV TVC Goose Flight Controller -> UAV TVC Goose II: Flight Controller
Changed lines of the file:
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@@
 	(paper "A4")
 	(title_block
-		(title "UAV TVC Goose Flight Controller")
+		(title "UAV TVC Goose II: Flight Controller")
 		(date "2024-08-05")
 		(rev "V2.1")
