File: hardware/flight-controller/power.kicad_sch (KiCad schematic)
At the start: 30 parts, among them J1 XT-60, Q1 IRFR5305, SW1 SW_Push_SPDT, U1 INA226, U2 LM1117MP-3.3, U3 VL14340

Commit message: Mouser
Parts:
- D1: value ~ -> SK56
- SW1: value SW_Push_SPDT -> JS102011SAQN
- U3: value VL14340 -> LV14340
Changed lines of the file:
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@@
 	(title_block
 		(title "UAV TVC Goose Flight Controller")
-		(date "2024-07-28")
+		(date "2024-07-31")
 		(rev "V2.1")
 		(comment 4 "Author: Eryk Możdżeń")
@@
 			)
 		)
-		(property "Value" "~"
+		(property "Value" "SK56"
 			(at 71.12 129.2224 90)
 			(effects
@@
 			)
 		)
-		(property "Datasheet" "~"
+		(property "Datasheet" "https://diotec.com/request/datasheet/sk52.pdf"
 			(at 73.66 128.27 0)
 			(effects
@@
 			)
 		)
-		(property "Value" "VL14340"
+		(property "Value" "LV14340"
 			(at 52.07 113.03 0)
 			(effects
@@
 			)
 		)
-		(property "Datasheet" "~"
+		(property "Datasheet" "https://www.mouser.pl/datasheet/2/447/pulse_plei_s_a0006349355_1-2904706.pdf"
 			(at 78.74 123.19 0)
 			(effects
@@
 		(dnp no)
 		(property "Reference" "SW1"
-			(at 58.166 71.12 90)
+			(at 54.102 69.85 90)
 			(effects
 				(font
 					(size 1.27 1.27)
 				)
-				(justify left)
+				(justify right)
 			)
 		)
-		(property "Value" "SW_Push_SPDT"
-			(at 44.45 72.3899 90)
+		(property "Value" "JS102011SAQN"
+			(at 54.102 71.882 90)
 			(effects
 				(font
 					(size 1.27 1.27)
 				)
-				(justify left)
-				(hide yes)
+				(justify right)
 			)
 		)
@@
 			)
 		)
-		(property "Datasheet" "~"
+		(property "Datasheet" "https://www.mouser.pl/datasheet/2/240/js-3050885.pdf"
 			(at 49.53 71.12 0)
 			(effects

Commit message: generate schematic in pdf
Other:
- title: UAV TVC Goose Flight Controller -> UAV TVC Goose II: Flight Controller
Changed lines of the file:
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@@
 	(paper "A4")
 	(title_block
-		(title "UAV TVC Goose Flight Controller")
+		(title "UAV TVC Goose II: Flight Controller")
 		(date "2024-08-05")
 		(rev "V2.1")
