File: hardware/flow-adapter/flow-adapter.kicad_pcb (KiCad board)
At the start: 2 copper layers, 40.5 x 24 mm, 7 parts, among them J1 IDC-10, J2 Conn_01x07

Commit message: new gerbers
Other:
- board text added: "JLCJLCJLCJLC"
Changed lines of the file:
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@@
 			(outputformat 1)
 			(mirror no)
-			(drillshape 1)
+			(drillshape 0)
 			(scaleselection 1)
-			(outputdirectory "")
+			(outputdirectory "gerbers/")
 		)
 	)
@@
 		)
 	)
+	(gr_text "JLCJLCJLCJLC"
+		(at 160.5 105.75 90)
+		(layer "F.SilkS")
+		(effects
+			(font
+				(size 1 1)
+				(thickness 0.15)
+			)
+			(justify left bottom)
+		)
+	)
