File: hardware/range-adapter/range-adapter.kicad_pcb (KiCad board)
At the start: 2 copper layers, 36.5 x 20.5 mm, 11 parts, among them J1 Conn_01x04, J2 IDC-10, U1 NTS0102

Commit message: new gerbers
Other:
- board text added: "JLCJLCJLCJLC"
Changed lines of the file:
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@@
 			(outputformat 1)
 			(mirror no)
-			(drillshape 1)
+			(drillshape 0)
 			(scaleselection 1)
-			(outputdirectory "")
+			(outputdirectory "gerbers/")
 		)
 	)
@@
 		(tags "capacitor")
 		(property "Reference" "C1"
-			(at 0 -1.429998 360)
+			(at 0 -1.429998 0)
 			(layer "F.SilkS")
 			(hide yes)
@@
 		)
 		(property "Value" "10u"
-			(at 0 1.429998 360)
+			(at 0 1.429998 0)
 			(layer "F.Fab")
 			(effects
@@
 		)
 		(fp_text user "${REFERENCE}"
-			(at 0 0 360)
+			(at 0 0 0)
 			(layer "F.Fab")
 			(effects
@@
 		(tags "capacitor")
 		(property "Reference" "C6"
-			(at 0 -1.429998 360)
+			(at 0 -1.429998 0)
 			(layer "F.SilkS")
 			(hide yes)
@@
 		)
 		(property "Value" "100n"
-			(at 0 1.429998 360)
+			(at 0 1.429998 0)
 			(layer "F.Fab")
 			(effects
@@
 		)
 		(fp_text user "${REFERENCE}"
-			(at 0 0 360)
+			(at 0 0 0)
 			(layer "F.Fab")
 			(effects
@@
 		(tags "capacitor")
 		(property "Reference" "C4"
-			(at 0 -1.429998 360)
+			(at 0 -1.429998 0)
 			(layer "F.SilkS")
 			(hide yes)
@@
 		)
 		(property "Value" "10u"
-			(at 0 1.429998 360)
+			(at 0 1.429998 0)
 			(layer "F.Fab")
 			(effects
@@
 		)
 		(fp_text user "${REFERENCE}"
-			(at 0 0 360)
+			(at 0 0 0)
 			(layer "F.Fab")
 			(effects
@@
 		(tags "capacitor")
 		(property "Reference" "C3"
-			(at 0 -1.429998 360)
+			(at 0 -1.429998 0)
 			(layer "F.SilkS")
 			(hide yes)
@@
 		)
 		(property "Value" "100n"
-			(at 0 1.429998 360)
+			(at 0 1.429998 0)
 			(layer "F.Fab")
 			(effects
@@
 		)
 		(fp_text user "${REFERENCE}"
-			(at 0 0 360)
+			(at 0 0 0)
 			(layer "F.Fab")
 			(effects
@@
 		(tags "capacitor")
 		(property "Reference" "C2"
-			(at 0 -1.429998 360)
+			(at 0 -1.429998 0)
 			(layer "F.SilkS")
 			(hide yes)
@@
 		)
 		(property "Value" "10u"
-			(at 0 1.429998 360)
+			(at 0 1.429998 0)
 			(layer "F.Fab")
 			(effects
@@
 		)
 		(fp_text user "${REFERENCE}"
-			(at 0 0 360)
+			(at 0 0 0)
 			(layer "F.Fab")
 			(effects
@@
 		(tags "capacitor")
 		(property "Reference" "C5"
-			(at 0 -1.429998 360)
+			(at 0 -1.429998 0)
 			(layer "F.SilkS")
 			(hide yes)
@@
 		)
 		(property "Value" "10u"
-			(at 0 1.429998 360)
+			(at 0 1.429998 0)
 			(layer "F.Fab")
 			(effects
@@
 		)
 		(fp_text user "${REFERENCE}"
-			(at 0 0 360)
+			(at 0 0 0)
 			(layer "F.Fab")
 			(effects
@@
 		)
 	)
+	(gr_text "JLCJLCJLCJLC"
+		(at 194.25 105 90)
+		(layer "F.SilkS")
+		(effects
+			(font
+				(size 1 1)
+				(thickness 0.15)
+			)
+			(justify left bottom)
+		)
+	)
