File: hardware/tachometer/tachometer.kicad_pcb (KiCad board)
At the start: 2 copper layers, 26 x 20 mm, 18 parts, among them J1 IDC-10, U1 CS49E, U2 NTS0102, U3 LM393

Commit message: new gerbers
Other:
- board text added: "JLCJLCJLCJLC"
Changed lines of the file:
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@@
 			(outputformat 1)
 			(mirror no)
-			(drillshape 1)
+			(drillshape 0)
 			(scaleselection 1)
-			(outputdirectory "")
+			(outputdirectory "gerbers/")
 		)
 	)
@@
 		(tags "resistor")
 		(property "Reference" "R2"
-			(at 0 1.429998 360)
+			(at 0 1.429998 0)
 			(layer "B.SilkS")
 			(hide yes)
@@
 		)
 		(property "Value" "100k"
-			(at 0 -1.429998 360)
+			(at 0 -1.429998 0)
 			(layer "B.Fab")
 			(effects
@@
 		)
 		(fp_text user "${REFERENCE}"
-			(at 0 0 360)
+			(at 0 0 0)
 			(layer "B.Fab")
 			(effects
@@
 		(tags "resistor")
 		(property "Reference" "R5"
-			(at 0 1.649998 360)
+			(at 0 1.649998 0)
 			(layer "B.SilkS")
 			(hide yes)
@@
 		)
 		(property "Value" "220k"
-			(at 0 -1.649998 360)
+			(at 0 -1.649998 0)
 			(layer "B.Fab")
 			(effects
@@
 		)
 		(fp_text user "${REFERENCE}"
-			(at 0 0 360)
+			(at 0 0 0)
 			(layer "B.Fab")
 			(effects
@@
 		(tags "resistor")
 		(property "Reference" "R1"
-			(at 0 1.649998 360)
+			(at 0 1.649998 0)
 			(layer "B.SilkS")
 			(hide yes)
@@
 		)
 		(property "Value" "100k"
-			(at 0 -1.649998 360)
+			(at 0 -1.649998 0)
 			(layer "B.Fab")
 			(effects
@@
 		)
 		(fp_text user "${REFERENCE}"
-			(at 0 0 360)
+			(at 0 0 0)
 			(layer "B.Fab")
 			(effects
@@
 		(tags "resistor")
 		(property "Reference" "R4"
-			(at 0 1.649998 360)
+			(at 0 1.649998 0)
 			(layer "B.SilkS")
 			(hide yes)
@@
 		)
 		(property "Value" "1k5"
-			(at 0 -1.649998 360)
+			(at 0 -1.649998 0)
 			(layer "B.Fab")
 			(effects
@@
 		)
 		(fp_text user "${REFERENCE}"
-			(at 0 0 360)
+			(at 0 0 0)
 			(layer "B.Fab")
 			(effects
@@
 		(tags "resistor")
 		(property "Reference" "R3"
-			(at 0 1.649998 360)
+			(at 0 1.649998 0)
 			(layer "B.SilkS")
 			(hide yes)
@@
 		)
 		(property "Value" "200k"
-			(at 0 -1.649998 360)
+			(at 0 -1.649998 0)
 			(layer "B.Fab")
 			(effects
@@
 		)
 		(fp_text user "${REFERENCE}"
-			(at 0 0 360)
+			(at 0 0 0)
 			(layer "B.Fab")
 			(effects
@@
 		)
 	)
+	(gr_text "JLCJLCJLCJLC"
+		(at 205.75 104.25 90)
+		(layer "F.SilkS")
+		(effects
+			(font
+				(size 1 1)
+				(thickness 0.15)
+			)
+			(justify left bottom)
+		)
+	)
